File: Library/Design_Blocks/Dinginator.kicad_blocks/USB C 2.0.kicad_block/USB C 2.0.kicad_sch (KiCad schematic)
At the start: 5 parts, among them J1 USB_C_Receptacle_USB2.0, U4 TPD4E1U06DCKR

Commit message: Progress?
Parts:
- renumbered D2 to D1, R9 to R1, R10 to R2, U4 to U1
Other:
- removed sheet RP2040
- removed sheet Solenoid Driver
- note removed: "LiPo powered Rp2040 MCU Rust firmware 2 plus solenoids? 1A min bidirectional solenoid driving"
- note removed: "Measure Vbat? USB for RP2040 filtering cap for input? charging and protection for cell? Power latch to be able to power down if flat from micro?"
- moved on the sheet: D1, J1, R1, R2, U1
